File: pcb/m47Board-C0/m47Board-C0.kicad_sch (KiCad schematic)
At the start: 28 parts, among them J1 Conn_01x05, J2 Conn_01x10, J3 Conn_01x10, J4 Conn_01x10, J5 Conn_01x10, J6 Conn_01x02, SW1 SW_Push, SW2 SW_Push, U1 TLV1117LV, U2 STM32C031C6Tx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

Commit message: Add R values
Parts:
- R1, R2, R3: value R -> 1k
Other:
- title: m47BoardV0 -> m47Board-C0
Changed lines of the file:
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@@
 	(paper "A4")
 	(title_block
-		(title "m47BoardV0")
+		(title "m47Board-C0")
 	)
 	(text "MCU"
@@
 			)
 		)
-		(property "Value" "R"
+		(property "Value" "1k"
 			(at 204.47 50.7999 0)
 			(show_name no)
@@
 			)
 		)
-		(property "Value" "R"
+		(property "Value" "1k"
 			(at 74.93 168.9099 0)
 			(show_name no)
@@
 			)
 		)
-		(property "Value" "R"
+		(property "Value" "1k"
 			(at 43.18 167.6399 0)
 			(show_name no)
