File: pcb/m47Board-H503/m47Board-H503.kicad_sch (KiCad schematic)
At the start: 41 parts, among them J1 USB_C_Receptacle_USB2.0_14P, J2 Conn_01x05_Pin, J3 Conn_01x10_Pin, J4 Conn_01x10_Pin, J5 Conn_01x10_Pin, J6 Conn_01x10_Pin, SW1 SW_Push, SW2 SW_Push, SW3 SW_Push, U1 AP2114H-3.3TRG1, U2 STM32H503CBTx, Y1 16MHz, Y2 Crystal_GND24

Commit message: Add USB-C ESD protection to m47Board-H503 schematic
Parts:
- added C11: 100n, symbol Device:C
- added D2: SMAJ5.0A, Diode_SMD:D_SMA, symbol Diode:SMAJ5.0A
- added U3: USBLC6-2SC6, Package_TO_SOT_SMD:SOT-23-6, symbol Power_Protection:USBLC6-2SC6
- renumbered C11 to C12, C12 to C13, C13 to C14, C14 to C15, C15 to C16, C16 to C17, C17 to C18, D2 to D3, R4 to R2, R5 to R3, R2 to R4, R3 to R5
Connections:
- net GND: now also R4.2, R5.2, C11.2, D2.2 (A2), U3.2 (GND); no longer R4.1, R5.1
- net USB_D+: now also U3.6 (I/O1); no longer J1.A6 (D+), J1.B6 (D+)
- net USB_D-: now also U3.4 (I/O2); no longer J1.A7 (D-), J1.B7 (D-)
- net VBUS: now also C11.1, D2.1 (A1), U3.5 (VBUS)
- net USB-C-CC2: now reaches J1.B5 (CC2)
- net USB-C-CC2: now also R5.1; no longer R5.2
- net USB-C-CC1: now reaches J1.A5 (CC1)
- net USB-C-CC1: now also R4.1; no longer R4.2
- new net: J1.A6 (D+), J1.B6 (D+), U3.1 (I/O1)
- new net: J1.A7 (D-), J1.B7 (D-), U3.3 (I/O2)
Other:
- note added: "C11 close to USBLC6"
- moved on the sheet: J1, R4, R5

Commit message: Add footprints to m47Board-H503 schematic
Parts:
- removed Y2: Crystal_GND24, symbol Device:Crystal_GND24
- added Y2: ABS07-32.768KHZ-T, Crystal:Crystal_SMD_3215-2Pin_3.2x1.5mm, symbol Device:Crystal
- C1, C12, C13, C7, C8, C9: footprint (none) -> Capacitor_SMD:C_0805_2012Metric_Pad1.18x1.45mm_HandSolder
- C10, C11, C14, C15, C18, C2, C3, C4, C5, C6: footprint (none) -> Capacitor_SMD:C_0603_1608Metric_Pad1.08x0.95mm_HandSolder
- C16, C17: value C -> 5.1p; footprint (none) -> Capacitor_SMD:C_0603_1608Metric_Pad1.08x0.95mm_HandSolder
- D1, D3: footprint (none) -> LED_SMD:LED_0603_1608Metric_Pad1.05x0.95mm_HandSolder
- J1: footprint (none) -> Connector_USB:USB_C_Receptacle_GCT_USB4105-xx-A_16P_TopMnt_Horizontal
- J2: footprint (none) -> Connector_PinHeader_2.54mm:PinHeader_1x05_P2.54mm_Vertical
- J3, J4, J5, J6: footprint (none) -> Connector_PinHeader_2.54mm:PinHeader_1x10_P2.54mm_Vertical
- R1, R2, R3, R4, R5, R6, R7, R8, R9: footprint (none) -> Resistor_SMD:R_0603_1608Metric_Pad0.98x0.95mm_HandSolder
- SW1, SW2, SW3: footprint (none) -> Button_Switch_SMD:SW_Push_1P1T_NO_E-Switch_TL3301NxxxxxG
- Y1: value 16MHz -> CX3225FB16000F0FZZH1 16MHz; footprint (none) -> Crystal:Crystal_SMD_3225-4Pin_3.2x2.5mm
Connections:
- net PC14: now also Y2.1
- net PC15: now also Y2.2
Other:
- note added: "(C_Load - C_stray)*2 C_load = 10p C_stray = [3;5]p"
- note added: "C values from ST recomendations"
- note removed: "(C_Load - C_stray)*2 C_load = 10p C_stray = 5p"

Commit message: Start making m47Board-H503 PCB layout
Parts:
- C10, C11, C14, C15, C16, C17, C18, C2, C3, C4, C5, C6: footprint Capacitor_SMD:C_0603_1608Metric_Pad1.08x0.95mm_HandSolder -> Capacitor_SMD:C_0402_1005Metric_Pad0.74x0.62mm_HandSolder
- D1, D3: footprint LED_SMD:LED_0603_1608Metric_Pad1.05x0.95mm_HandSolder -> LED_SMD:LED_0805_2012Metric_Pad1.15x1.40mm_HandSolder
- R1, R2, R3, R4, R5, R6, R7, R8, R9: footprint Resistor_SMD:R_0603_1608Metric_Pad0.98x0.95mm_HandSolder -> Resistor_SMD:R_0402_1005Metric_Pad0.72x0.64mm_HandSolder
Connections:
- net USB_D+: now also U3.1 (I/O1); no longer U3.6 (I/O1)
- net USB_D-: now also U3.3 (I/O2); no longer U3.4 (I/O2)
- net at J1.A6 (D+), J1.B6 (D+): now also U3.6 (I/O1); no longer U3.1 (I/O1)
- net at J1.A7 (D-), J1.B7 (D-): now also U3.4 (I/O2); no longer U3.3 (I/O2)

Commit message: m47Board-H503 PCB layout update
Parts:
- removed J5, J6: Conn_01x10_Pin, Connector_PinHeader_2.54mm:PinHeader_1x10_P2.54mm_Vertical, symbol Connector:Conn_01x10_Pin
- added J5: Conn_01x09_Pin, Connector_PinHeader_2.54mm:PinHeader_1x09_P2.54mm_Vertical, symbol Connector:Conn_01x09_Pin
- added J6: Conn_01x06_Pin, Connector_PinHeader_2.54mm:PinHeader_1x06_P2.54mm_Vertical, symbol Connector:Conn_01x06_Pin
Other:
- moved on the sheet: R6, R7

Commit message: m47Board-H503 PCB layout update
Parts:
- removed J2: Conn_01x05_Pin, Connector_PinHeader_2.54mm:PinHeader_1x05_P2.54mm_Vertical, symbol Connector:Conn_01x05_Pin
- removed J3: Conn_01x10_Pin, Connector_PinHeader_2.54mm:PinHeader_1x10_P2.54mm_Vertical, symbol Connector:Conn_01x10_Pin
- removed J5: Conn_01x09_Pin, Connector_PinHeader_2.54mm:PinHeader_1x09_P2.54mm_Vertical, symbol Connector:Conn_01x09_Pin
- removed J6: Conn_01x06_Pin, Connector_PinHeader_2.54mm:PinHeader_1x06_P2.54mm_Vertical, symbol Connector:Conn_01x06_Pin
- added J3, J5: Conn_01x15_Pin, Connector_PinHeader_2.54mm:PinHeader_1x15_P2.54mm_Vertical, symbol Connector:Conn_01x15_Pin
Connections:
- net +3.3V: now also J3.1 (Pin_1)
- net GND: now also J3.3 (Pin_3)
- net NRST: now also J3.5 (Pin_5)
- net SWCLK: now also J3.2 (Pin_2)
- net SWDIO: now also J3.4 (Pin_4)
Other:
- moved on the sheet: R6, R7
